File: OtherFiles/Laboratorio 2/emitter follower.sch (EAGLE design)
At the start: 4 parts

Commit message: continuato analisi laboratorio 2
Connections:
- removed net -10V: RE.1
- net GND: now also RE.1
Changed lines of the file:
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@@
 <part name="GND1" library="supply1" library_urn="urn:adsk.eagle:library:371" deviceset="GND" device=""/>
 <part name="SUPPLY1" library="supply2" library_urn="urn:adsk.eagle:library:372" deviceset="+10V" device=""/>
-<part name="SUPPLY2" library="supply2" library_urn="urn:adsk.eagle:library:372" deviceset="-10V" device=""/>
+<part name="GND2" library="supply1" library_urn="urn:adsk.eagle:library:371" deviceset="GND" device=""/>
 </parts>
 <sheets>
@@
 </instance>
 <instance part="VI" gate="G$1" x="27.94" y="30.48" smashed="yes">
-<attribute name="NAME" x="35.56" y="30.48" size="1.778" layer="95"/>
+<attribute name="NAME" x="34.036" y="30.734" size="1.778" layer="95"/>
 </instance>
 <instance part="RE" gate="G$1" x="55.88" y="25.4" smashed="yes" rot="R90">
@@
 <attribute name="VALUE" x="53.34" y="61.595" size="1.778" layer="96"/>
 </instance>
-<instance part="SUPPLY2" gate="G$1" x="55.88" y="15.24" smashed="yes">
-<attribute name="VALUE" x="52.705" y="10.541" size="1.778" layer="96"/>
+<instance part="GND2" gate="1" x="55.88" y="15.24" smashed="yes">
+<attribute name="VALUE" x="53.34" y="12.7" size="1.778" layer="96"/>
 </instance>
 </instances>
@@
 <wire x1="27.94" y1="22.86" x2="27.94" y2="17.78" width="0.1524" layer="91"/>
 </segment>
+<segment>
+<pinref part="RE" gate="G$1" pin="1"/>
+<wire x1="55.88" y1="17.78" x2="55.88" y2="20.32" width="0.1524" layer="91"/>
+<pinref part="GND2" gate="1" pin="GND"/>
+</segment>
 </net>
 <net name="+10V" class="0">
@@
 </segment>
 </net>
-<net name="-10V" class="0">
-<segment>
-<pinref part="RE" gate="G$1" pin="1"/>
-<wire x1="55.88" y1="17.78" x2="55.88" y2="20.32" width="0.1524" layer="91"/>
-<pinref part="SUPPLY2" gate="G$1" pin="-10V"/>
-</segment>
-</net>
